File: kicad/pmt-control.kicad_pcb (KiCad board)
At the start: 2 copper layers, 91.4 x 66 mm, 27 parts, among them J1 OUT, Q1 2N7000, Q2 2N7000, SW1 Rotary_Encoder_Switch, SW2 TTL, SW3 RST, U1 Pico, U2 AD5761BRUZ-AD5761BRUZ, U3 MAX6951, U4 LM285Z-2.5

Commit message: Finished board layout
Parts:
- moved D1 53.7 mm to (131.1, 98.6)
- moved R1 52.5 mm to (98.0, 60.7)
- moved C1 51.1 mm to (131.8, 80.8)
- moved R4 49.2 mm to (131.8, 84.1)
- moved Q2 45.9 mm to (131.1, 93.7)
- moved R3 45.8 mm to (138.2, 98.6), turned to 180 degrees
- moved U4 44.4 mm to (133.3, 68.6), turned to 270 degrees
- moved C4 17.9 mm to (103.1, 92.2)
- moved Q1 16.0 mm to (122.2, 93.7)
- moved U2 0.25 mm to (123.4, 82.5)
Routing:
- net Net-(U1-Pad4): track 0.00 -> 122.4 mm, vias 0 -> 1
- net +5V: track 0.00 -> 120.9 mm, vias 0 -> 2
- net Net-(U1-Pad7): track 0.00 -> 93.3 mm
- net Net-(U1-Pad6): track 0.00 -> 92.5 mm
- net Net-(U1-Pad5): track 0.00 -> 92.4 mm
- net Net-(R1-Pad2): track 0.00 -> 72.4 mm, vias 0 -> 1
- net Net-(SW1-PadA): track 0.00 -> 63.3 mm
- net GND: track 37.2 -> 92.7 mm, vias 0 -> 2
- net Net-(SW1-PadB): track 0.00 -> 55.1 mm
- net MISO: track 0.00 -> 45.2 mm, vias 0 -> 2
- net +3V3: track 19.0 -> 64.0 mm, vias 0 -> 3
- net Net-(Q1-Pad1): track 0.00 -> 41.3 mm, vias 0 -> 1
- net SCK: track 18.7 -> 56.0 mm, vias 0 -> 2
- net MOSI: track 15.4 -> 50.3 mm, vias 0 -> 2
- net Net-(J1-Pad3): track 0.00 -> 21.6 mm
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